File: HARDWARE/PCB/EAGLE/esp32_logging.brd (EAGLE design)
At the start: 92.9 x 48.3 mm, 100 parts, among them IC1 LM2596SX-5.0_NOPB, IC12 EL357, IC2 EL357, IC3 EL357, IC5 M3406-ADJ, IC6 DW01A, J2 1803277, J3 1803280, J4 1803280, J5 1803277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

Commit message: FEAT: add rs485 line
Parts:
- added C19, C2: 100nf, SamacSys_Parts:CAPC1608X87N
- added D22, D23: TISP4240M3BJR-S, TISP4240M3BJR-S:TISP4240M3BJRS
- added D6: SM712-02HTG, SamacSys_Parts:SOT95P237X111-3N
- added F3, F4: 1206L010_60WR, 1206L010_60WR:1206L075132WR
- added IC22: ISL83483IBZ, ISL83483IBZ:SOIC127P600X175-8N
- added J1: 1803277, AccesControlNFC:1803277
- added R40: 10k, AccesControlNFC:RESC1608X55N
- added R42: 120, SamacSys_Parts:RESC2012X65N
- added R60, R61: 47, SamacSys_Parts:RESC1608X55N
- moved EXT 18.1 mm to (23.1, 49.0)
- moved SW1 0.38 mm to (37.8, 30.1)
Connections:
- removed net 19: ESP32.14
- removed net 20: ESP32.13
- new net A: D6.1, F3.2, IC22.6
- new net A_OUT: D23.1, F3.1, J1.1, R42.2
- new net B: D6.2, F4.2, IC22.7
- new net B_OUT: D22.1, F4.1, J1.2, R42.1
- new net N$62: IC22.1, R61.2
- new net N$95: IC22.4, R60.2
- new net RE/DE: IC22.2, IC22.3, R40.2
- new net RX_RS485: ESP32.16, R61.1
- new net TX_RS485: ESP32.27, R60.1
- net 3.3V: now also C19.2, C2.2, IC22.8, R40.1
- net GND: now also C19.1, C2.1, D22.2, D23.2, D6.3, IC22.5
- net IN_D2: now also ESP32.13; no longer ESP32.27
- net IN_D3: now also ESP32.14; no longer ESP32.16
Routing:
- net 3.3V: track 226.0 -> 274.4 mm, vias 7 -> 8
- net B: track 0.00 -> 26.5 mm
- net A: track 0.00 -> 16.6 mm
- net IN_D2: track 44.1 -> 29.0 mm
- net TX_RS485: track 0.00 -> 12.9 mm, vias 0 -> 1
- net A_OUT: track 0.00 -> 11.6 mm
- net B_OUT: track 0.00 -> 11.1 mm
- net SDA: track 48.1 -> 59.0 mm, vias 4 -> 3
- net RE/DE: track 0.00 -> 7.96 mm
- net GND: track 35.9 -> 43.1 mm
- net IN_D3: track 37.3 -> 30.4 mm
- net RX_RS485: track 0.00 -> 6.16 mm, vias 0 -> 1
- net MOSI: track 90.4 -> 87.4 mm
- net N$62: track 0.00 -> 2.58 mm
- net CS_SDCARD: track 46.3 -> 43.8 mm
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Other:
- board text added: "A"
- board text added: "B"
- board text added: "ESP32 LOGGING V1.1"
- board text added: "POSITRON ELEKTRONIK"
- board text removed: "ESP32_LOGGING v1.0"
- board text removed: "POSITRON ELECTRONIC"
