File: HARDWARE/PCB/EAGLE/esp32_logging.sch (EAGLE design)
At the start: 100 parts, among them IC1 LM2596SX-5.0_NOPB, IC12 EL357, IC2 EL357, IC3 EL357, IC5 M3406-ADJ, IC6 DW01A, J2 1803277, J3 1803280, J4 1803280, J5 1803277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

Commit message: FEAT: add rs485 line
Parts:
- added C19, C2: 100nf, SamacSys_Parts:885012206071
- added D22, D23: TISP4240M3BJR-S, TISP4240M3BJR-S:TISP4240M3BJR-S
- added D6: SM712-02HTG, SamacSys_Parts:SM712-02HTG
- added F3, F4: 1206L010_60WR, 1206L010_60WR:1206L010_60WR
- added IC22: ISL83483IBZ, ISL83483IBZ:ISL83483IBZ
- added J1: 1803277, AccesControlNFC:1803277
- added R40: 10k, AccesControlNFC:ESR03EZPJ103
- added R42: 120, SamacSys_Parts:ESR10EZPJ121
- added R60, R61: 47, SamacSys_Parts:ERJ-PA3J470V
Connections:
- removed net 19: ESP32.IO12
- removed net 20: ESP32.IO14
- new net A: D6.TVS1, F3.2, IC22.A/Y
- new net A_OUT: D23.1, F3.1, J1.1, R42.2
- new net B: D6.TVS2, F4.2, IC22.B/Z
- new net B_OUT: D22.1, F4.1, J1.2, R42.1
- new net N$62: IC22.RO, R61.2
- new net N$95: IC22.DI, R60.2
- new net RE/DE: IC22.!RE, IC22.DE, R40.2
- new net RX_RS485: ESP32.IO13, R61.1
- new net TX_RS485: ESP32.IO16, R60.1
- net 3.3V: now also C19.2, C2.2, IC22.VCC, R40.1
- net GND: now also C19.1, C2.1, D22.2, D23.2, D6.COMMON, IC22.GND
- net IN_D2: now also ESP32.IO14; no longer ESP32.IO16
- net IN_D3: now also ESP32.IO12; no longer ESP32.IO13
Other:
- note added: "RS485"
- note added: "Regulator 3V3 Batt Charger RS485 DI and DO"
- note removed: "Regulator 3V3 Batt Charger DI and DO"
